Commit message: Moved camera

File: manta_description/urdf/sensors.xacro (robot description, xacro)
@@ -17,5 +17,5 @@
   <!-- Mount a camera  -->
   <xacro:default_camera namespace="${namespace}" parent_link="${namespace}/base_link" suffix="front">
-    <origin xyz="0.30 0 0" rpy="0 0 0"/>
+    <origin xyz="0.26 0 0.01" rpy="0 0 0"/>
   </xacro:default_camera>
 </robot>
