Commit message: Modified inertia

File: manta_description/urdf/base.xacro (robot description, xacro)
@@ -12,5 +12,5 @@
     Vehicle's parameters (remember to enter the model parameters below)
   -->
-  <xacro:property name="mass" value="24.52"/>
+  <xacro:property name="mass" value="18.8"/>
   <!-- Center of gravity -->
   <xacro:property name="cog" value="0 0 0"/>
@@ -39,7 +39,7 @@
           <mass value="${mass}" />
           <origin xyz="${cog}" rpy="0 0 0"/>
-          <inertia ixx="0" ixy="0" ixz="0"
-                   iyy="0" iyz="0"
-                   izz="0" />
+          <inertia ixx="${438.5}" ixy="${0.0}" ixz="${0.0}"
+            iyy="${438.5}" iyz="${0.0}" izz="${811.0}" />
+	<!--<inertia ixx="${0.503217}" ixy="${0.000204}" ixz="${-0.000526}" iyy="${0.493449}" iyz="${0.000038}" izz="${0.919819}" /> -->
         </inertial>
         <visual>
@@ -48,5 +48,4 @@
             <mesh filename="${visual_mesh_file}" scale="0.001 0.001 0.001" />
           </geometry>
-          <color rgba="0 1.0 1.0 1.0"/>
         </visual>
         <collision>

File: manta_description/urdf/gazebo.xacro (robot description, xacro)
@@ -4,5 +4,5 @@
     <xacro:property name="manta_cob" value="0 0 0.05"/>
     <!-- Vehicle's actual volume (Gazebo cannot compute the volume out of the mesh) -->
-    <xacro:property name="manta_volume" value="0.024"/>
+    <xacro:property name="manta_volume" value="0.019"/>
     <!-- Describing the dimensions of the vehicle's bounding box -->
     <xacro:property name="manta_length" value="0.63"/>
@@ -36,18 +36,20 @@
         <hydrodynamic_model>
           <type>fossen</type>
+          <!-- Added mass: see p.28 in Berg2012 -->
           <added_mass>
-            1 0 0 0 0 0
-            0 1 0 0 0 0
-            0 0 1 0 0 0
-            0 0 0 1 0 0
-            0 0 0 0 1 0
-            0 0 0 0 0 1
+            10.7727 0 0 0 0 0
+            0 10.7727 0 0 0 0
+            0 0 49.7679 0 0 0
+            0 0 0 1.0092 0 0
+            0 0 0 0 1.0092 0
+            0  0  0  0  0  0
           </added_mass>
           <!--
             The linear damping coefficients can be provided as a diagonal (6 elements)
             or a full matrix (36 coefficients), like the added-mass coefficients above
+            Linear damping: see p.31 in Berg2012
           -->
           <linear_damping>
-            0 0 0 0 0 0
+            -19.5909 -19.5909 -50.5595 -13.3040 -13.2181 -1.1559
           </linear_damping>
           <!--
@@ -57,13 +59,14 @@
             This matrix is mostly useful for slender bodies (e.g. AUVs with torpedo shape)
           -->
-          <linear_damping_forward_speed>
+          <!-- <linear_damping_forward_speed>
             0 0 0 0 0 0
-          </linear_damping_forward_speed>
+          </linear_damping_forward_speed> -->
           <!--
             The quadratic damping coefficients can be provided as a diagonal (6 elements)
             or a full matrix (36 coefficients), like the added-mass coefficients above
+            Non-linear damping: see p.30 in Berg2012
           -->
           <quadratic_damping>
-            0 0 0 0 0 0
+            -5.1386 -5.1386 -26.1105 0 0 0
           </quadratic_damping>
           <!--
